File: MCU/MCU/ExternalInput.sch (KiCad schematic (older format))
At the start: 25 parts, among them J14 Conn_01x02, J15 Conn_01x02, J16 Conn_01x02, J17 Conn_01x04, J18 Conn_01x02, U15 LMV321, U16 MAX3232

Commit message: MCU routed
Parts:
- removed FB4: 1K, Resistors_SMD:R_0805, symbol Device:Ferrite_Bead_Small
- added D25: SD103, lc_lib:SOD-123, symbol MySchLib:D_Schottky_Small
Connections:
- net GND: no longer C53.2, J17.4 (Pin_4)
- net GNDD: now also C53.2, J17.4 (Pin_4)
- net PTT_RTS: now also D25.2 (K)
- net at J17.1 (Pin_1): now also D25.1 (A)
Changed lines of the file:
@@
 	0    -1   -1   0
-$EndComp
-$Comp
-L power:GND #PWR?
-U 1 1 5EA99E44
-P 2000 2600
-AR Path="/5E7D94C5/5EA99E44" Ref="#PWR?"  Part="1"
-AR Path="/5EA95119/5EA99E44" Ref="#PWR095"  Part="1"
-F 0 "#PWR095" H 2000 2350 50  0001 C CNN
-F 1 "GND" H 2005 2427 50  0000 C CNN
-F 2 "" H 2000 2600 50  0001 C CNN
-F 3 "" H 2000 2600 50  0001 C CNN
-	1    2000 2600
-	1    0    0    -1
 $EndComp
 Wire Wire Line
@@
 Text Notes 1750 2150 0    50   ~ 0
 TX GND
-$Comp
-L power:GND #PWR?
-U 1 1 5F1D7559
-P 3050 2600
-AR Path="/5E7D94C5/5F1D7559" Ref="#PWR?"  Part="1"
-AR Path="/5EA95119/5F1D7559" Ref="#PWR098"  Part="1"
-F 0 "#PWR098" H 3050 2350 50  0001 C CNN
-F 1 "GND" H 3055 2427 50  0000 C CNN
-F 2 "" H 3050 2600 50  0001 C CNN
-F 3 "" H 3050 2600 50  0001 C CNN
-	1    3050 2600
-	1    0    0    -1
-$EndComp
 Text HLabel 2400 3050 3    50   Output ~ 0
 PTT_RTS
@@
 Wire Wire Line
 	5050 4900 5050 4800
-$Comp
-L power:GND #PWR?
-U 1 1 5E41AEF8
-P 4750 5000
-AR Path="/5E7D94C5/5E41AEF8" Ref="#PWR?"  Part="1"
-AR Path="/5EA95119/5E41AEF8" Ref="#PWR0125"  Part="1"
-F 0 "#PWR0125" H 4750 4750 50  0001 C CNN
-F 1 "GND" H 4755 4827 50  0000 C CNN
-F 2 "" H 4750 5000 50  0001 C CNN
-F 3 "" H 4750 5000 50  0001 C CNN
-	1    4750 5000
-	1    0    0    -1
-$EndComp
 Wire Wire Line
 	4750 5000 4750 4900
@@
 	0    -1   1    0
 $EndComp
-$Comp
-L Device:Ferrite_Bead_Small FB4
-U 1 1 5E498DD9
-P 2400 2850
-F 0 "FB4" H 2500 2896 50  0000 L CNN
-F 1 "1K" H 2500 2805 50  0000 L CNN
-F 2 "Resistors_SMD:R_0805" V 2330 2850 50  0001 C CNN
-F 3 "~" H 2400 2850 50  0001 C CNN
-	1    2400 2850
-	1    0    0    -1
-$EndComp
 Wire Wire Line
 	2400 2750 2400 2650
@@
 Wire Wire Line
 	2250 6000 2350 6000
+$Comp
+L power:GNDD #PWR0146
+U 1 1 5E65BD42
+P 3050 2600
+F 0 "#PWR0146" H 3050 2350 50  0001 C CNN
+F 1 "GNDD" H 3054 2445 50  0000 C CNN
+F 2 "" H 3050 2600 50  0001 C CNN
+F 3 "" H 3050 2600 50  0001 C CNN
+	1    3050 2600
+	1    0    0    -1
+$EndComp
+$Comp
+L power:GND #PWR?
+U 1 1 5E65D41A
+P 2000 2600
+AR Path="/5E7D94C5/5E65D41A" Ref="#PWR?"  Part="1"
+AR Path="/5EA95119/5E65D41A" Ref="#PWR0148"  Part="1"
+F 0 "#PWR0148" H 2000 2350 50  0001 C CNN
+F 1 "GND" H 2005 2427 50  0000 C CNN
+F 2 "" H 2000 2600 50  0001 C CNN
+F 3 "" H 2000 2600 50  0001 C CNN
+	1    2000 2600
+	1    0    0    -1
+$EndComp
+$Comp
+L power:GNDD #PWR0149
+U 1 1 5E65E6DB
+P 4750 5000
+F 0 "#PWR0149" H 4750 4750 50  0001 C CNN
+F 1 "GNDD" H 4754 4845 50  0000 C CNN
+F 2 "" H 4750 5000 50  0001 C CNN
+F 3 "" H 4750 5000 50  0001 C CNN
+	1    4750 5000
+	1    0    0    -1
+$EndComp
+$Comp
+L MySchLib:D_Schottky_Small D?
+U 1 1 5E520B7E
+P 2400 2850
+AR Path="/5E7D94C5/5E520B7E" Ref="D?"  Part="1"
+AR Path="/5EA95119/5E520B7E" Ref="D25"  Part="1"
+F 0 "D25" V 2446 2782 50  0000 R CNN
+F 1 "SD103" V 2355 2782 50  0000 R CNN
+F 2 "lc_lib:SOD-123" V 2400 2850 50  0001 C CNN
+F 3 "~" V 2400 2850 50  0001 C CNN
+	1    2400 2850
+	0    -1   -1   0
+$EndComp
 $EndSCHEMATC

Commit message: Power module
Parts:
- added C60: 104, Capacitors_SMD:C_0805, symbol Device:C_Small
- added J20: CAN, Connectors_JST:JST_XH_B02B-XH-A_02x2.50mm_Straight, symbol Connector_Generic:Conn_01x02
- added R85, R86: 100, Resistors_SMD:R_0805, symbol Device:R_Small
- added R87: 120, Resistors_SMD:R_0805, symbol Device:R_Small
- added U17: TJA1042T, lc_lib:SOIC-8_150MIL, symbol Interface_CAN_LIN:TJA1042T
Connections:
- net GND: now also C60.1, U17.2 (GND), U17.8 (STB)
- new net: R85.1, U17.1 (TXD)
- new net: R86.1, U17.4 (RXD)
- new net +5VA: C60.2, U17.3 (VCC)
- new net CAN+: J20.2 (Pin_2), R87.1, U17.7 (CANH)
- new net CAN-: J20.1 (Pin_1), R87.2, U17.6 (CANL)
- new net CAN_RX: R86.2
- new net CAN_TX: R85.2
Changed lines of the file:
@@
 	0    -1   -1   0
 $EndComp
+$Comp
+L Connector_Generic:Conn_01x02 J20
+U 1 1 5E54ECE3
+P 5900 2150
+F 0 "J20" V 5864 2230 50  0000 L CNN
+F 1 "CAN" V 5773 2230 50  0000 L CNN
+F 2 "Connectors_JST:JST_XH_B02B-XH-A_02x2.50mm_Straight" H 5900 2150 50  0001 C CNN
+F 3 "~" H 5900 2150 50  0001 C CNN
+	1    5900 2150
+	0    1    -1   0
+$EndComp
+$Comp
+L Interface_CAN_LIN:TJA1042T U17
+U 1 1 5E54FC2A
+P 5850 3350
+F 0 "U17" V 5896 2906 50  0000 R CNN
+F 1 "TJA1042T" V 5805 2906 50  0000 R CNN
+F 2 "lc_lib:SOIC-8_150MIL" H 5850 2850 50  0001 C CIN
+F 3 "http://www.nxp.com/documents/data_sheet/TJA1042.pdf" H 5850 3350 50  0001 C CNN
+	1    5850 3350
+	0    -1   -1   0
+$EndComp
+$Comp
+L Device:R_Small R87
+U 1 1 5E551309
+P 5850 2650
+F 0 "R87" H 5909 2696 50  0000 L CNN
+F 1 "120" H 5909 2605 50  0000 L CNN
+F 2 "Resistors_SMD:R_0805" H 5850 2650 50  0001 C CNN
+F 3 "~" H 5850 2650 50  0001 C CNN
+	1    5850 2650
+	0    -1   -1   0
+$EndComp
+Wire Wire Line
+	5750 2850 5750 2650
+Wire Wire Line
+	5750 2650 5750 2450
+Wire Wire Line
+	5750 2450 5800 2450
+Wire Wire Line
+	5800 2450 5800 2350
+Connection ~ 5750 2650
+Wire Wire Line
+	5900 2350 5900 2450
+Wire Wire Line
+	5900 2450 5950 2450
+Wire Wire Line
+	5950 2450 5950 2650
+Wire Wire Line
+	5950 2650 5950 2850
+Connection ~ 5950 2650
+Wire Wire Line
+	5250 3300 5250 3350
+Wire Wire Line
+	5250 3350 5450 3350
+$Comp
+L Device:C_Small C60
+U 1 1 5E55CC73
+P 5250 3500
+F 0 "C60" V 5350 3500 50  0000 C CNN
+F 1 "104" V 5400 3500 50  0000 C CNN
+F 2 "Capacitors_SMD:C_0805" H 5250 3500 50  0001 C CNN
+F 3 "~" H 5250 3500 50  0001 C CNN
+	1    5250 3500
+	-1   0    0    1
+$EndComp
+Wire Wire Line
+	5250 3400 5250 3350
+Connection ~ 5250 3350
+$Comp
+L power:GND #PWR?
+U 1 1 5E55F53A
+P 5250 3650
+AR Path="/5E7D94C5/5E55F53A" Ref="#PWR?"  Part="1"
+AR Path="/5EA95119/5E55F53A" Ref="#PWR0155"  Part="1"
+F 0 "#PWR0155" H 5250 3400 50  0001 C CNN
+F 1 "GND" H 5255 3477 50  0000 C CNN
+F 2 "" H 5250 3650 50  0001 C CNN
+F 3 "" H 5250 3650 50  0001 C CNN
+	1    5250 3650
+	1    0    0    -1
+$EndComp
+Wire Wire Line
+	5250 3650 5250 3600
+$Comp
+L power:GND #PWR?
+U 1 1 5E561C2E
+P 6350 3400
+AR Path="/5E7D94C5/5E561C2E" Ref="#PWR?"  Part="1"
+AR Path="/5EA95119/5E561C2E" Ref="#PWR0156"  Part="1"
+F 0 "#PWR0156" H 6350 3150 50  0001 C CNN
+F 1 "GND" H 6355 3227 50  0000 C CNN
+F 2 "" H 6350 3400 50  0001 C CNN
+F 3 "" H 6350 3400 50  0001 C CNN
+	1    6350 3400
+	1    0    0    -1
+$EndComp
+Wire Wire Line
+	6350 3400 6350 3350
+Wire Wire Line
+	6350 3350 6250 3350
+Text HLabel 5650 4100 3    50   Input ~ 0
+CAN_TX
+Text HLabel 5800 4250 3    50   Output ~ 0
+CAN_RX
+Wire Wire Line
+	5800 4250 5800 4200
+Wire Wire Line
+	5800 4200 5750 4200
+$Comp
+L power:GND #PWR?
+U 1 1 5E56A7E1
+P 6050 3950
+AR Path="/5E7D94C5/5E56A7E1" Ref="#PWR?"  Part="1"
+AR Path="/5EA95119/5E56A7E1" Ref="#PWR0157"  Part="1"
+F 0 "#PWR0157" H 6050 3700 50  0001 C CNN
+F 1 "GND" H 6055 3777 50  0000 C CNN
+F 2 "" H 6050 3950 50  0001 C CNN
+F 3 "" H 6050 3950 50  0001 C CNN
+	1    6050 3950
+	1    0    0    -1
+$EndComp
+Wire Wire Line
+	6050 3850 6050 3950
+$Comp
+L Device:R_Small R85
+U 1 1 5E56E527
+P 5650 3950
+F 0 "R85" H 5709 3996 50  0000 L CNN
+F 1 "100" H 5709 3905 50  0000 L CNN
+F 2 "Resistors_SMD:R_0805" H 5650 3950 50  0001 C CNN
+F 3 "~" H 5650 3950 50  0001 C CNN
+	1    5650 3950
+	1    0    0    -1
+$EndComp
+Wire Wire Line
+	5650 4050 5650 4100
+$Comp
+L Device:R_Small R86
+U 1 1 5E56E9EE
+P 5750 4100
+F 0 "R86" H 5809 4146 50  0000 L CNN
+F 1 "100" H 5809 4055 50  0000 L CNN
+F 2 "Resistors_SMD:R_0805" H 5750 4100 50  0001 C CNN
+F 3 "~" H 5750 4100 50  0001 C CNN
+	1    5750 4100
+	1    0    0    -1
+$EndComp
+Wire Wire Line
+	5750 3850 5750 4000
+Text GLabel 5700 2450 0    50   Input ~ 0
+CAN+
+Wire Wire Line
+	5700 2450 5750 2450
+Connection ~ 5750 2450
+Text GLabel 6000 2450 2    50   Input ~ 0
+CAN-
+Wire Wire Line
+	6000 2450 5950 2450
+Connection ~ 5950 2450
+$Comp
+L power:+5VA #PWR?
+U 1 1 5E65814C
+P 5250 3300
+F 0 "#PWR?" H 5250 3150 50  0001 C CNN
+F 1 "+5VA" H 5265 3473 50  0000 C CNN
+F 2 "" H 5250 3300 50  0001 C CNN
+F 3 "" H 5250 3300 50  0001 C CNN
+	1    5250 3300
+	1    0    0    -1
+$EndComp
 $EndSCHEMATC
