File: MCU/MCU/MCU.kicad_pcb (KiCad board)
At the start: 2 copper layers, 130 x 100 mm, 236 parts, among them J1 Conn_01x08, J10 Conn_01x02, J11 Conn_01x02, J12 Conn_01x02, J13 Conn_01x02, J14 Conn_01x02, J15 Conn_01x02, J16 Conn_01x02, J17 Conn_01x04, J18 Conn_01x02, J19 Conn_01x02, J2 Conn_01x08, J3 Conn_02x20_Odd_Even, J4 Conn_01x04, J5 Conn_01x04, J6 Conn_01x02, J7 Conn_01x02, J8 Conn_01x06, J9 Conn_01x06, M1 Fan, M2 Fan, Q1 8050, Q10 AO3402, Q11 AO3402, Q2 8050, Q3 8050, Q4 8550, Q5 8050, Q6 8050, Q7 8050, Q8 8550, Q9 8050, U1 74HC04, U10 LMV321, U11 PC817, U12 SY8303, U13 AZ1117-3.3, U14 AZ1117-3.3, U15 LMV321, U16 MAX3232, U2 STM32F407VETx, U3 LMV324, U4 LMV324, U5 LMV358, U6 LMV324, U7 LMV324, U8 LMV321, U9 ICL7660, Y1 12MHz

Commit message: routing
Parts:
- moved D24 74.1 mm to (65.5, 85.0), turned to 135 degrees
- moved R84 62.9 mm to (64.0, 86.5), turned to 315 degrees
- moved C3 27.6 mm to (66.0, 53.0), turned to 135 degrees
- moved C42 3.55 mm to (45.5, 27.5)
- moved C43 3.55 mm to (52.0, 28.5)
- moved C44 3.55 mm to (57.0, 29.2)
- moved C45 3.55 mm to (56.0, 25.0)
- moved C47 3.55 mm to (58.0, 25.0)
- moved C49 3.55 mm to (63.0, 37.8)
- moved D22 3.55 mm to (63.8, 25.0)
- moved D8 3.55 mm to (40.8, 31.0)
- moved L4 3.55 mm to (41.0, 27.0)
- moved L5 3.55 mm to (51.9, 25.2)
- moved R63 3.55 mm to (46.0, 31.5)
- moved R64 3.55 mm to (51.2, 37.0)
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Routing:
- net +3V3: track 105.0 -> 380.8 mm, vias 2 -> 14
- net /ADC1_5: track 0.00 -> 119.7 mm, vias 0 -> 4
- net /ADC1_9: track 0.00 -> 115.9 mm
- net /ADC1_14: track 0.00 -> 111.4 mm, vias 0 -> 2
- net /ADC1_6: track 0.00 -> 110.5 mm, vias 0 -> 2
- net /ADC1_8: track 0.00 -> 106.7 mm, vias 0 -> 2
- net /ADC1_7: track 0.00 -> 103.7 mm, vias 0 -> 2
- net /ADC1_4: track 0.00 -> 102.3 mm, vias 0 -> 2
- net /ADC1_3: track 0.00 -> 98.5 mm, vias 0 -> 2
- net +12V: track 0.00 -> 94.3 mm
- net ALC_trig: track 2.63 -> 95.4 mm, vias 1 -> 4
- net +5V: track 0.00 -> 90.7 mm, vias 0 -> 2
- net Net-(D1-Pad2): track 0.00 -> 84.8 mm, vias 0 -> 10
- net VBL: track 0.00 -> 79.3 mm, vias 0 -> 2
- net Transmit: track 4.84 -> 77.7 mm, vias 1 -> 4
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- added copper zone on B.Cu, net (none)
- added copper zone on B.Cu, net +12V
- added copper zone on B.Cu, net +3V3
- added copper zone on B.Cu, net +5V
- added copper zone on B.Cu, net GND
- added copper zone on B.Cu, net Net-(C41-Pad1)
- added copper zone on B.Cu, net Net-(C43-Pad1)
- added copper zone on B.Cu, net Net-(F1-Pad1)
- added copper zone on B.Cu, net VBL

Commit message: MCU routed
Parts:
- removed FB4: 1K, Resistors_SMD:R_0805
- added D25: SD103, lc_lib:SOD-123, B.Cu at (67.8, 111.2)
- added FB7: GND, Resistors_SMD:R_1206, B.Cu at (66.8, 43.0)
- F1: value 1A -> 3A
- L4: value 22uH -> BEAD
- moved R59 1.50 mm to (120.8, 57.0)
- moved C5 1.25 mm to (68.7, 75.6)
- moved Q9 1.00 mm to (115.8, 61.8)
- moved C8 0.71 mm to (62.1, 81.3)
- moved Q1 0.30 mm to (71.9, 116.5)
- moved D15 0.25 mm to (125.2, 59.8)
- moved R58 0.25 mm to (120.4, 60.8)
- turned C36 to 90 degrees
- turned D8 to 0 degrees
Connections:
- C10 pad 2: GNDA -> GND
- C11 pad 2: GNDA -> GND
- C13 pad 2: GNDA -> GND
- C14 pad 2: GNDA -> GND
- C15 pad 2: GNDA -> GND
- C16 pad 2: GNDA -> GND
- C17 pad 2: GNDA -> GND
- C18 pad 2: GNDA -> GND
- C19 pad 2: GNDA -> GND
- C20 pad 2: GNDA -> GND
- C21 pad 2: GNDA -> GND
- C22 pad 2: GNDA -> GND
- C23 pad 2: GNDA -> GND
- C24 pad 2: GNDA -> GND
- C25 pad 2: GNDA -> GND
- C26 pad 2: GNDA -> GND
- C27 pad 2: GNDA -> GND
- C28 pad 2: GNDA -> GND
- C29 pad 2: GNDA -> GND
- C30 pad 2: GNDA -> GND
- C31 pad 2: GNDA -> GND
- C32 pad 2: GNDA -> GND
- C36 pad 1: Net-(C36-Pad1) -> GND
- C36 pad 2: GND -> Net-(C36-Pad2)
- C53 pad 2: GND -> GNDD
- C59 pad 2: GNDA -> GND
- D8 pad 1: +12V -> GND
- D8 pad 2: GND -> +12V
- J10 pad 2: GNDA -> GND
- J17 pad 4: GND -> GNDD
- J4 pad 4: GND -> GNDD
- J5 pad 4: GNDA -> GND
- J6 pad 2: GNDA -> GND
- J7 pad 2: GNDA -> GND
- J8 pad 1: GNDA -> GND
- J9 pad 1: GNDA -> GND
- R17 pad 1: GNDA -> GND
- R20 pad 1: GNDA -> GND
- R22 pad 1: GNDA -> GND
- R25 pad 1: GNDA -> GND
- R28 pad 1: GNDA -> GND
- R30 pad 1: GNDA -> GND
- R41 pad 1: GNDA -> GND
- R45 pad 2: Net-(C36-Pad1) -> Net-(C36-Pad2)
- RV1 pad 3: GNDA -> GND
- U2 pad 20: GNDA -> GND
- U3 pad 11: GNDA -> GND
- U4 pad 11: GNDA -> GND
- U5 pad 4: GNDA -> GND
- U6 pad 11: GNDA -> GND
- U7 pad 11: GNDA -> GND
- U8 pad 2: GNDA -> GND
- U9 pad 5: Net-(C36-Pad1) -> Net-(C36-Pad2)
Routing:
- net +12V: track 94.3 -> 304.8 mm, vias 0 -> 12
- net +3V3: track 380.8 -> 524.3 mm, vias 14 -> 30
- net PTT: track 0.00 -> 127.0 mm, vias 0 -> 8
- net /ADC3_0: track 5.36 -> 127.4 mm, vias 1 -> 6
- net +5V: track 90.7 -> 210.7 mm, vias 2 -> 6
- net /ADC3_13: track 16.6 -> 117.4 mm, vias 3 -> 6
- net /ADC3_12: track 17.5 -> 118.0 mm, vias 3 -> 6
- net SEL2: track 0.00 -> 95.7 mm, vias 0 -> 6
- net SEL3: track 0.00 -> 95.2 mm, vias 0 -> 6
- net SEL1: track 0.00 -> 94.4 mm, vias 0 -> 5
- net SEL6: track 0.00 -> 92.0 mm, vias 0 -> 6
- net SEL5: track 0.00 -> 90.7 mm, vias 0 -> 6
- net SEL4: track 0.00 -> 88.7 mm, vias 0 -> 6
- net SW_Bypass: track 0.00 -> 83.5 mm, vias 0 -> 4
- net GND: track 67.5 -> 147.2 mm, vias 50 -> 147
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- added copper zone on F.Cu, net GND
- added copper zone on B.Cu, net GNDD
- added copper zone on F.Cu, net GNDD
Other:
- board text added: "+"
- board text added: "+12V"
- board text added: "1"
- board text added: "12V"
- board text added: "2"
- board text added: "3"
- board text added: "4"
- board text added: "5"
- board text added: "6"
- board text added: "A"
- board text added: "ALC"
- board text added: "Band"
- board text added: "FUSE 3A"
- board text added: "Fan1"
- board text added: "Fan2"
- board text added: "GND"
- board text added: "Imain HIGH"
- board text added: "LPF"
- board text added: "MCU"
- board text added: "NTC1"
- board text added: "NTC2"
- board text added: "OPA1000 Control Board Rev 0.1 By Lu, Zening (BI4WOP) Feb. 14 2020"
- board text added: "Overdrive"
- board text added: "PWR Lim"
- board text added: "PWR Sense"
- board text added: "Power"
- board text added: "R"
- board text added: "REL In"
- board text added: "REL Out"
- board text added: "REVPWR 1 HIGH"
- board text added: "REVPWR2 HIGH"
- board text added: "RF Level"
- board text added: "RS232"
- board text added: "RTS"
- board text added: "Rotary Band Selector"
- board text added: "SW Bypass"
- board text added: "SW PWR"
- board text added: "SWR1"
- board text added: "SWR2"
- board text added: "T"
- board text added: "T1H"
- board text added: "T2H"
- board text added: "TFT: TK040F1532"
- board text added: "TX GND"
- board text added: "Upper-left"
- board text added: "Vmain HIGH"

Commit message: Power module
Parts:
- added C60: 104, Capacitors_SMD:C_0805, B.Cu at (32.8, 107.0)
- added J20: CAN, Connectors_JST:JST_XH_B02B-XH-A_02x2.50mm_Straight, B.Cu at (41.5, 117.2)
- added R82: 10K, Resistors_SMD:R_0805, B.Cu at (112.8, 69.8)
- added R83: 10K, Resistors_SMD:R_0805, B.Cu at (112.8, 67.8)
- added R85: 100, Resistors_SMD:R_0805, B.Cu at (28.8, 108.0)
- added R86: 100, Resistors_SMD:R_0805, B.Cu at (36.8, 108.0)
- added R87: 120, Resistors_SMD:R_0805, B.Cu at (33.0, 116.2)
- added U17: TJA1042T, lc_lib:SOIC-8_150MIL, B.Cu at (33.0, 111.6)
- J19: value Conn_01x02 -> Barrel_Jack_Switch; footprint Connectors_JST:JST_XH_B02B-XH-A_02x2.50mm_Straight -> Connectors:BARREL_JACK
- Q6: value 8050 -> 8550
- R54: value 47K -> 1K
- R55: value 100K -> 10
- moved F1 5.37 mm to (37.0, 31.2)
- moved J19 4.61 mm to (32.5, 28.8), turned to 270 degrees
- moved Q6 3.49 mm to (109.3, 68.0), turned to 270 degrees
- moved D8 1.27 mm to (42.0, 31.2)
- moved FB6 0.40 mm to (63.2, 111.5)
- moved D19 0.25 mm to (117.5, 75.0)
- moved FB5 0.15 mm to (60.0, 111.5)
Connections:
- net Net-(C48-Pad1) renamed +5VA
- Q6 pad 1: PWR_on_sig -> Net-(Q6-Pad1)
- Q6 pad 2: SW_PWR -> +3V3
- Q6 pad 3: PWR_on -> Net-(Q6-Pad3)
- Q7 pad 3: PWR_on_sig -> PWR_on
- R54 pad 1: +3V3 -> PWR_on_sig
- R54 pad 2: PWR_on -> Net-(Q6-Pad1)
- R55 pad 1: PWR_on_sig -> SW_PWR
- R55 pad 2: SW_PWR -> PWR_on
- U2 pad 51: Net-(U2-Pad51) -> /CAN_RX
- U2 pad 52: Net-(U2-Pad52) -> /CAN_TX
Routing:
- net +5VA: track 45.9 -> 130.4 mm, vias 0 -> 2
- net /CAN_RX: track 0.00 -> 63.2 mm, vias 0 -> 4
- net /CAN_TX: track 0.00 -> 62.2 mm, vias 0 -> 4
- net CAN+: track 0.00 -> 16.4 mm
- net +12V: track 304.8 -> 291.8 mm
- net CAN-: track 0.00 -> 13.0 mm
- net PWR_on_sig: track 69.0 -> 59.8 mm
- net +3V3: track 524.3 -> 532.2 mm, vias 30 -> 32
- net GND: track 147.2 -> 152.6 mm, vias 147 -> 149
- net Net-(Q6-Pad1): track 0.00 -> 3.92 mm
- net Net-(Q6-Pad3): track 0.00 -> 3.11 mm
- net GNDD: track 41.3 -> 38.2 mm, vias 76 -> 71
- net PWR_on: track 65.6 -> 68.7 mm
- net /TX: track 115.0 -> 117.8 mm
- net Net-(R85-Pad1): track 0.00 -> 2.48 mm
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- added copper zone on F.Cu, net Net-(C41-Pad1)
- removed copper zone on B.Cu, net +12V
- removed copper zone on B.Cu, net Net-(F1-Pad1)
