File: MCU/MCU/Power.sch (KiCad schematic (older format))
At the start: 44 parts, among them J19 Conn_01x02, M1 Fan, M2 Fan, Q10 AO3402, Q11 AO3402, U12 SY8303, U13 AZ1117-3.3, U14 AZ1117-3.3

Commit message: MCU routed
Parts:
- added FB7: GND, Resistors_SMD:R_1206, symbol Device:Ferrite_Bead_Small
- D8: symbol Device:D_Zener -> MySchLib:D_Zener
- F1: value 1A -> 3A
- L4: value 22uH -> BEAD
Connections:
- net +12V: now also D8.2 (K); no longer D8.1 (K)
- net GND: now also D8.1 (A), FB7.1; no longer D8.2 (A)
- new net GNDD: FB7.2
Changed lines of the file:
@@
 	1200 1650 1400 1650
 $Comp
-L Device:D_Zener D8
+L MySchLib:D_Zener D8
 U 1 1 5E220FED
 P 1600 2300
@@
 P 1200 1950
 F 0 "F1" V 1003 1950 50  0000 C CNN
-F 1 "1A" V 1094 1950 50  0000 C CNN
+F 1 "3A" V 1094 1950 50  0000 C CNN
 F 2 "Resistors_SMD:R_1206" V 1130 1950 50  0001 C CNN
 F 3 "~" H 1200 1950 50  0001 C CNN
@@
 P 1550 1650
 F 0 "L4" V 1775 1650 50  0000 C CNN
-F 1 "22uH" V 1684 1650 50  0000 C CNN
+F 1 "BEAD" V 1684 1650 50  0000 C CNN
 F 2 "Inductors_SMD:L_1206" H 1550 1650 50  0001 C CNN
 F 3 "~" H 1550 1650 50  0001 C CNN
@@
 Wire Wire Line
 	4100 1100 4250 1100
+$Comp
+L Device:Ferrite_Bead_Small FB7
+U 1 1 5E4713FC
+P 3750 5950
+F 0 "FB7" V 3513 5950 50  0000 C CNN
+F 1 "GND" V 3604 5950 50  0000 C CNN
+F 2 "Resistors_SMD:R_1206" V 3680 5950 50  0001 C CNN
+F 3 "~" H 3750 5950 50  0001 C CNN
+	1    3750 5950
+	0    1    1    0
+$EndComp
+$Comp
+L power:GND #PWR0150
+U 1 1 5E472F1D
+P 4050 6050
+F 0 "#PWR0150" H 4050 5800 50  0001 C CNN
+F 1 "GND" H 4055 5877 50  0000 C CNN
+F 2 "" H 4050 6050 50  0001 C CNN
+F 3 "" H 4050 6050 50  0001 C CNN
+	1    4050 6050
+	1    0    0    -1
+$EndComp
+$Comp
+L power:GNDA #PWR0151
+U 1 1 5E473989
+P 4300 6050
+F 0 "#PWR0151" H 4300 5800 50  0001 C CNN
+F 1 "GNDA" H 4305 5877 50  0000 C CNN
+F 2 "" H 4300 6050 50  0001 C CNN
+F 3 "" H 4300 6050 50  0001 C CNN
+	1    4300 6050
+	1    0    0    -1
+$EndComp
+Wire Wire Line
+	4300 6050 4300 5950
+Wire Wire Line
+	4300 5950 4050 5950
+Wire Wire Line
+	4050 6050 4050 5950
+Connection ~ 4050 5950
+Wire Wire Line
+	4050 5950 3850 5950
+$Comp
+L power:GNDD #PWR0152
+U 1 1 5E47C8AA
+P 3500 6150
+F 0 "#PWR0152" H 3500 5900 50  0001 C CNN
+F 1 "GNDD" H 3504 5995 50  0000 C CNN
+F 2 "" H 3500 6150 50  0001 C CNN
+F 3 "" H 3500 6150 50  0001 C CNN
+	1    3500 6150
+	1    0    0    -1
+$EndComp
+Wire Wire Line
+	3500 6150 3500 5950
+Wire Wire Line
+	3500 5950 3650 5950
 $EndSCHEMATC

Commit message: Power module
Parts:
- removed J19: Conn_01x02, Connectors_JST:JST_XH_B02B-XH-A_02x2.50mm_Straight, symbol Connector_Generic:Conn_01x02
- added J19: Barrel_Jack_Switch, Connectors:BARREL_JACK, symbol Connector:Barrel_Jack_Switch
Connections:
- net GND: now also J19.2, J19.3
- net at F1.1: now also J19.1
- net +5VA: now reaches C48.1, R71.1, U13.3 (VI), U14.3 (VI)
Changed lines of the file:
@@
 Wire Wire Line
 	1600 2450 1600 2650
-$Comp
-L Connector_Generic:Conn_01x02 J19
-U 1 1 5E2F3078
-P 900 2150
-F 0 "J19" H 818 2367 50  0000 C CNN
-F 1 "Conn_01x02" H 818 2276 50  0000 C CNN
-F 2 "Connectors_JST:JST_XH_B02B-XH-A_02x2.50mm_Straight" H 900 2150 50  0001 C CNN
-F 3 "~" H 900 2150 50  0001 C CNN
-	1    900  2150
-	-1   0    0    -1
-$EndComp
-Wire Wire Line
-	1100 2150 1200 2150
 Connection ~ 1200 1650
-Wire Wire Line
-	1100 2250 1200 2250
 $Comp
 L power:GND #PWR0102
@@
 	1    0    0    -1
 $EndComp
-Wire Wire Line
-	1200 2250 1200 2450
 $Comp
 L Device:C_Small C45
@@
 Wire Wire Line
 	3500 5950 3650 5950
+Wire Wire Line
+	1050 2350 1200 2350
+Wire Wire Line
+	1200 2350 1200 2450
+Wire Wire Line
+	1050 2150 1200 2150
+$Comp
+L Connector:Barrel_Jack_Switch J19
+U 1 1 5E52FEDF
+P 750 2250
+F 0 "J19" H 807 2567 50  0000 C CNN
+F 1 "Barrel_Jack_Switch" H 807 2476 50  0000 C CNN
+F 2 "Connectors:BARREL_JACK" H 800 2210 50  0001 C CNN
+F 3 "~" H 800 2210 50  0001 C CNN
+	1    750  2250
+	1    0    0    -1
+$EndComp
+Wire Wire Line
+	1050 2250 1200 2250
+Wire Wire Line
+	1200 2250 1200 2350
+Connection ~ 1200 2350
+$Comp
+L power:+5VA #PWR?
+U 1 1 5E65574F
+P 5300 1650
+F 0 "#PWR?" H 5300 1500 50  0001 C CNN
+F 1 "+5VA" H 5315 1823 50  0000 C CNN
+F 2 "" H 5300 1650 50  0001 C CNN
+F 3 "" H 5300 1650 50  0001 C CNN
+	1    5300 1650
+	1    0    0    -1
+$EndComp
 $EndSCHEMATC
