File: Interface2/interface.sch (KiCad schematic (older format))
At the start: 77 parts, among them J1 RS232 CAT, J10 AudioJack_PJ325, J2 DR9_Dual_Male, J3 CIV out, J4 AudioJack_PJ325, J5 RF sense, J6 AudioJack_PJ325, J7 ALC trig, J8 AudioJack_PJ325, J9 +3.3V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

Commit message: COM
Parts:
- removed C10, C15: 103, lc_lib:0805_C, symbol Device:C_Small
- removed C11: 20p, lc_lib:0805_C, symbol Device:C_Small
- removed C12: 102, lc_lib:0805_C, symbol Device:C_Small
- removed C14, C7: 104, lc_lib:0805_C, symbol Device:C_Small
- removed C16: 1uF, lc_lib:0805_C, symbol Device:C_Small
- removed C5: 104, lc_lib:1206_C, symbol Device:C_Small
- removed C6: 10uF, lc_lib:0805_C, symbol Device:C_Small
- removed C9: 10uF, lc_lib:1206_C, symbol Device:C_Small
- removed D5: 1N4148, lc_lib:LL-34, symbol MySchLib:D
- removed L6, L8: 1uH, lc_lib:0805_L, symbol Device:L
- removed R11, R12, R13, R3: 1K, lc_lib:0805_R, symbol Device:R_Small
- removed R14, R23: 0, lc_lib:0805_R, symbol Device:R_Small
- removed R15: 10k, lc_lib:0805_R, symbol Device:R_Small
- removed R6, R9: --, lc_lib:0805_R, symbol Device:R_Small
- removed R7: 2.2K, lc_lib:0805_R, symbol Device:R_Small
- removed R8: 100, lc_lib:0805_R, symbol Device:R_Small
- removed RV1: 10K, Potentiometers:Potentiometer_Trimmer_Bourns_3296W, symbol Device:R_POT
- removed U1: ICL7660, lc_lib:SOIC-8_150MIL, symbol Regulator_SwitchedCapacitor:ICL7660
- removed U2: LMV321, lc_lib:SOT-23-5, symbol Amplifier_Operational:LMV321
- removed U3: TL431, lc_lib:SOT-23(SOT-23-3), symbol MySchLib:TL431
- added R?: 1K, lc_lib:0805_R, symbol Device:R_Small
- C1, C2, C3: value 102 -> 100pF
- FB1: value Ferrite_Bead_Small -> 100
Connections:
- net labels removed: VRef
- wire segments 250 -> 166
Other:
- moved on the sheet: C17, C18, FB1, J9
