File: RF/OPA1000_RF/RF_input/RF_input.sch (KiCad schematic (older format))
At the start: 47 parts, among them J1 +12V, J2 GND, J3 In, Q1 BLF188XR, Q2 2N3904, SW1 SW_SPDT, T1 Transformer_4_1, U1 LM358, U2 TL431

Commit message: OPA1000 and 2000 compatibility
Parts:
- Q1: symbol MySchLib:BLF188XR -> RF_input-rescue:BLF188XR-MySchLib
Connections:
- net G1: now also Q1.3 (G)
- net G2: now also Q1.4 (G)
Other:
- moved on the sheet: C4, C6, C7, J3, Q1, R12, R13, R14, R15, R16, R17, R18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
